Commit message: urdf and xml for the new robotzel

File: biped_robot_description/urdf/robot_urdf_2023_02_20_v3.urdf (robot description, URDF)
Before this commit: robot biped, 14 links, 13 joints
Links:
- removed link L_FOOT_CONTACT
- removed link R_FOOT_CONTACT
- removed link imu
- link L_FOOT: geometry collision mesh filename=package://robot_urdf_2023_02_20_v3/meshes/L_FOOT.STL; visual mesh filename=package://robot_urdf_2023_02_20_v3/meshes/L_FOOT.STL
- link L_HIP: mass 0.0629568480892822 -> 0.0629568480892821; geometry collision mesh filename=package://robot_urdf_2023_02_20_v3/meshes/L_HIP.STL; visual mesh filename=package://robot_urdf_2023_02_20_v3/meshes/L_HIP.STL
- link L_LOWER_LEG: geometry collision mesh filename=package://robot_urdf_2023_02_20_v3/meshes/L_LOWER_LEG.STL; visual mesh filename=package://robot_urdf_2023_02_20_v3/meshes/L_LOWER_LEG.STL
- link L_SHOULDER: geometry collision mesh filename=package://robot_urdf_2023_02_20_v3/meshes/L_SHOULDER.STL; visual mesh filename=package://robot_urdf_2023_02_20_v3/meshes/L_SHOULDER.STL
- link L_UPPER_LEG: geometry collision mesh filename=package://robot_urdf_2023_02_20_v3/meshes/L_UPPER_LEG.STL; visual mesh filename=package://robot_urdf_2023_02_20_v3/meshes/L_UPPER_LEG.STL
- link R_FOOT: geometry collision mesh filename=package://robot_urdf_2023_02_20_v3/meshes/R_FOOT.STL; visual mesh filename=package://robot_urdf_2023_02_20_v3/meshes/R_FOOT.STL
- link R_HIP: geometry collision mesh filename=package://robot_urdf_2023_02_20_v3/meshes/R_HIP.STL; visual mesh filename=package://robot_urdf_2023_02_20_v3/meshes/R_HIP.STL
- link R_LOWER_LEG: geometry collision mesh filename=package://robot_urdf_2023_02_20_v3/meshes/R_LOWER_LEG.STL; visual mesh filename=package://robot_urdf_2023_02_20_v3/meshes/R_LOWER_LEG.STL
- link R_SHOULDER: geometry collision mesh filename=package://robot_urdf_2023_02_20_v3/meshes/R_SHOULDER.STL; visual mesh filename=package://robot_urdf_2023_02_20_v3/meshes/R_SHOULDER.STL
- link R_UPPER_LEG: geometry collision mesh filename=package://robot_urdf_2023_02_20_v3/meshes/R_UPPER_LEG.STL; visual mesh filename=package://robot_urdf_2023_02_20_v3/meshes/R_UPPER_LEG.STL
- link base_link: geometry collision mesh filename=package://robot_urdf_2023_02_20_v3/meshes/base_link.STL; visual mesh filename=package://robot_urdf_2023_02_20_v3/meshes/base_link.STL
Joints:
- removed joint L_FOOT_CONTACT_JOINT
- removed joint R_FOOT_CONTACT_JOINT
- removed joint imu_joint
- joint L_KFE: limit lower=-2.2 upper=-0.1 effort=1000 velocity=1000 -> lower=-2.2 upper=-0.1 effort=1000 velocity=0
- joint R_ANKLE: origin xyz=0 0.0173 -0.30826 rpy=0 0 0 -> xyz=0 0.0168 -0.30826 rpy=0 0 0
