Commit message: fix urdf mesh resource path

File: biped_robot_description/urdf/custom_robot.urdf (robot description, URDF)
Before this commit: robot biped, 11 links, 10 joints
Links:
- link FL_FOOT: geometry collision mesh filename=package://biped_robot_description/meshes/FL_FOOT.STL
- link FL_HIP: geometry collision mesh filename=package://biped_robot_description/meshes/FL_HIP.STL; visual mesh filename=package://biped_robot_description/meshes/FL_HIP.STL
- link FL_LOWER_LEG: geometry collision mesh filename=package://biped_robot_description/meshes/FL_LOWER_LEG.STL; visual mesh filename=package://biped_robot_description/meshes/FL_LOWER_LEG.STL
- link FL_SHOULDER: geometry collision mesh filename=package://biped_robot_description/meshes/FL_SHOULDER.STL; visual mesh filename=package://biped_robot_description/meshes/FL_SHOULDER.STL
- link FL_UPPER_LEG: geometry collision mesh filename=package://biped_robot_description/meshes/FL_UPPER_LEG.STL; visual mesh filename=package://biped_robot_description/meshes/FL_UPPER_LEG.STL
- link FR_FOOT: geometry collision mesh filename=package://biped_robot_description/meshes/FR_FOOT.STL
- link FR_HIP: geometry collision mesh filename=package://biped_robot_description/meshes/FR_HIP.STL; visual mesh filename=package://biped_robot_description/meshes/FR_HIP.STL
- link FR_LOWER_LEG: geometry collision mesh filename=package://biped_robot_description/meshes/FR_LOWER_LEG.STL; visual mesh filename=package://biped_robot_description/meshes/FR_LOWER_LEG.STL
- link FR_SHOULDER: geometry collision mesh filename=package://biped_robot_description/meshes/FR_SHOULDER.STL; visual mesh filename=package://biped_robot_description/meshes/FR_SHOULDER.STL
- link FR_UPPER_LEG: geometry collision mesh filename=package://biped_robot_description/meshes/FR_UPPER_LEG.STL; visual mesh filename=package://biped_robot_description/meshes/FR_UPPER_LEG.STL
- link base_link: geometry collision mesh filename=package://biped_robot_description/meshes/base_link.STL; visual mesh filename=package://biped_robot_description/meshes/base_link.STL

Commit message: fix urdf limits

File: biped_robot_description/urdf/custom_robot.urdf (robot description, URDF)
Before this commit: robot biped, 11 links, 10 joints
Joints:
- joint FL_ANKLE: limit lower=0 upper=0 effort=0 velocity=0 -> lower=-10 upper=10 effort=1000 velocity=1000
- joint FL_KFE: limit lower=0 upper=0 effort=0 velocity=0 -> lower=-10 upper=10 effort=1000 velocity=1000
- joint FR_ANKLE: limit lower=0 upper=0 effort=0 velocity=0 -> lower=-10 upper=10 effort=1000 velocity=1000
- joint FR_KFE: limit lower=0 upper=0 effort=0 velocity=0 -> lower=-10 upper=10 effort=1000 velocity=1000

Commit message: add urdf feet visual

File: biped_robot_description/urdf/custom_robot.urdf (robot description, URDF)
Before this commit: robot biped, 11 links, 10 joints
Links:
- link FL_FOOT: geometry collision mesh filename=package://biped_robot_description/meshes/FL_FOOT.STL; visual mesh filename=package://biped_robot_description/meshes/FL_FOOT.STL
- link FR_FOOT: geometry collision mesh filename=package://biped_robot_description/meshes/FR_FOOT.STL; visual mesh filename=package://biped_robot_description/meshes/FR_FOOT.STL

Commit message: fix urdf joint orientations, disable yaw joint

File: biped_robot_description/urdf/custom_robot.urdf (robot description, URDF)
Before this commit: robot biped, 11 links, 10 joints
Joints:
- joint FL_HAA: axis 1 0 0 -> -1 0 0
- joint FL_HFE: axis 0 1 0 -> 0 -1 0
- joint FL_KFE: axis 0 1 0 -> 0 -1 0
- joint FL_YAW: type revolute -> fixed
- joint FR_HAA: axis 1 0 0 -> -1 0 0
- joint FR_YAW: type revolute -> fixed

Commit message: fix axis direction and joint

File: biped_robot_description/urdf/custom_robot.urdf (robot description, URDF)
Before this commit: robot biped, 11 links, 10 joints
Joints:
- joint FL_HAA: axis -1 0 0 -> 1 0 0
- joint FL_HFE: axis 0 -1 0 -> 0 1 0
- joint FL_KFE: axis 0 -1 0 -> 0 1 0
- joint FL_YAW: type fixed -> revolute
- joint FR_YAW: type fixed -> revolute

Commit message: fix axis direction

File: biped_robot_description/urdf/custom_robot.urdf (robot description, URDF)
Before this commit: robot biped, 11 links, 10 joints
Joints:
- joint FR_HAA: axis -1 0 0 -> 1 0 0

Commit message: urdf joint limits

File: biped_robot_description/urdf/custom_robot.urdf (robot description, URDF)
Before this commit: robot biped, 11 links, 10 joints
Joints:
- joint FL_ANKLE: limit lower=-10 upper=10 effort=1000 velocity=1000 -> lower=-1.6 upper=1.6 effort=1000 velocity=1000
- joint FL_HAA: limit lower=-10 upper=10 effort=1000 velocity=1000 -> lower=-0.25 upper=0.25 effort=1000 velocity=1000
- joint FL_HFE: limit lower=-10 upper=10 effort=1000 velocity=1000 -> lower=-1.5 upper=1.5 effort=1000 velocity=1000
- joint FL_KFE: limit lower=-10 upper=10 effort=1000 velocity=1000 -> lower=-2.2 upper=2.2 effort=1000 velocity=1000
- joint FL_YAW: limit lower=-10 upper=10 effort=1000 velocity=1000 -> lower=-0.3 upper=0.3 effort=1000 velocity=1000
- joint FR_ANKLE: limit lower=-10 upper=10 effort=1000 velocity=1000 -> lower=-1.6 upper=1.6 effort=1000 velocity=1000
- joint FR_HAA: limit lower=-10 upper=10 effort=1000 velocity=1000 -> lower=-0.25 upper=0.25 effort=1000 velocity=1000
- joint FR_HFE: limit lower=-10 upper=10 effort=1000 velocity=1000 -> lower=-1.5 upper=1.5 effort=1000 velocity=1000
- joint FR_KFE: limit lower=-10 upper=10 effort=1000 velocity=1000 -> lower=-2.2 upper=2.2 effort=1000 velocity=1000
- joint FR_YAW: limit lower=-10 upper=10 effort=1000 velocity=1000 -> lower=-0.3 upper=0.3 effort=1000 velocity=1000

Commit message: change ik limit

File: biped_robot_description/urdf/custom_robot.urdf (robot description, URDF)
Before this commit: robot biped, 11 links, 10 joints
Joints:
- joint FL_KFE: limit lower=-2.2 upper=2.2 effort=1000 velocity=1000 -> lower=0.01 upper=2.2 effort=1000 velocity=1000
- joint FR_KFE: limit lower=-2.2 upper=2.2 effort=1000 velocity=1000 -> lower=0.01 upper=2.2 effort=1000 velocity=1000

Commit message: add imu sensor and limits

File: biped_robot_description/urdf/custom_robot.urdf (robot description, URDF)
Before this commit: robot biped, 11 links, 10 joints
Links:
- added link imu, mass 0.01; visual box size=0.03 0.03 0.01
Joints:
- added joint imu_joint: type fixed, parent base_link, child imu, origin xyz=0 0 0 rpy=-3.141592 0 0
- joint FL_KFE: limit lower=0.01 upper=2.2 effort=1000 velocity=1000 -> lower=-2.2 upper=-0.1 effort=1000 velocity=1000
- joint FR_KFE: limit lower=0.01 upper=2.2 effort=1000 velocity=1000 -> lower=-2.2 upper=-0.1 effort=1000 velocity=1000

Commit message: remove Front from the urdf

File: biped_robot_description/urdf/custom_robot.urdf (robot description, URDF)
Before this commit: robot biped, 12 links, 11 joints
Links:
- removed link FL_FOOT
- removed link FL_HIP
- removed link FL_LOWER_LEG
- removed link FL_SHOULDER
- removed link FL_UPPER_LEG
- removed link FR_FOOT
- removed link FR_HIP
- removed link FR_LOWER_LEG
- removed link FR_SHOULDER
- removed link FR_UPPER_LEG
- added link L_FOOT, mass 0.0001; collision mesh filename=package://biped_robot_description/meshes/L_FOOT.STL; visual mesh filename=package://biped_robot_description/meshes/L_FOOT.STL
- added link L_HIP, mass 0.01; collision mesh filename=package://biped_robot_description/meshes/L_HIP.STL; visual mesh filename=package://biped_robot_description/meshes/L_HIP.STL
- added link L_LOWER_LEG, mass 0.0911245737414644; collision mesh filename=package://biped_robot_description/meshes/L_LOWER_LEG.STL; visual mesh filename=package://biped_robot_description/meshes/L_LOWER_LEG.STL
- added link L_SHOULDER, mass 0.307022440099937; collision mesh filename=package://biped_robot_description/meshes/L_SHOULDER.STL; visual mesh filename=package://biped_robot_description/meshes/L_SHOULDER.STL
- added link L_UPPER_LEG, mass 0.459365803346259; collision mesh filename=package://biped_robot_description/meshes/L_UPPER_LEG.STL; visual mesh filename=package://biped_robot_description/meshes/L_UPPER_LEG.STL
- added link R_FOOT, mass 0.0001; collision mesh filename=package://biped_robot_description/meshes/R_FOOT.STL; visual mesh filename=package://biped_robot_description/meshes/R_FOOT.STL
- added link R_HIP, mass 0.35434; collision mesh filename=package://biped_robot_description/meshes/R_HIP.STL; visual mesh filename=package://biped_robot_description/meshes/R_HIP.STL
- added link R_LOWER_LEG, mass 0.0911245737715333; collision mesh filename=package://biped_robot_description/meshes/R_LOWER_LEG.STL; visual mesh filename=package://biped_robot_description/meshes/R_LOWER_LEG.STL
- added link R_SHOULDER, mass 0.30702; collision mesh filename=package://biped_robot_description/meshes/R_SHOULDER.STL; visual mesh filename=package://biped_robot_description/meshes/R_SHOULDER.STL
- added link R_UPPER_LEG, mass 0.459365802658862; collision mesh filename=package://biped_robot_description/meshes/R_UPPER_LEG.STL; visual mesh filename=package://biped_robot_description/meshes/R_UPPER_LEG.STL
Joints:
- removed joint FL_ANKLE
- removed joint FL_HAA
- removed joint FL_HFE
- removed joint FL_KFE
- removed joint FL_YAW
- removed joint FR_ANKLE
- removed joint FR_HAA
- removed joint FR_HFE
- removed joint FR_KFE
- removed joint FR_YAW
- added joint L_ANKLE: type revolute, parent L_LOWER_LEG, child L_FOOT, origin xyz=0 -0.0168 -0.30826 rpy=0 0 0, axis 0 1 0, limit lower=-1.6 upper=1.6 effort=1000 velocity=1000
- added joint L_HAA: type revolute, parent L_HIP, child L_SHOULDER, origin xyz=0 0 -0.073 rpy=0 0 0, axis 1 0 0, limit lower=-0.25 upper=0.25 effort=1000 velocity=1000
- added joint L_HFE: type revolute, parent L_SHOULDER, child L_UPPER_LEG, origin xyz=0 0 0 rpy=0 0 0, axis 0 1 0, limit lower=-1.5 upper=1.5 effort=1000 velocity=1000
- added joint L_KFE: type revolute, parent L_UPPER_LEG, child L_LOWER_LEG, origin xyz=0.0099993 0.0584 -0.23393 rpy=0 0 0, axis 0 1 0, limit lower=-2.2 upper=-0.1 effort=1000 velocity=1000
- added joint L_YAW: type revolute, parent base_link, child L_HIP, origin xyz=0 0.07 -0.0158 rpy=0 0 0, axis 0 0 1, limit lower=-0.3 upper=0.3 effort=1000 velocity=1000
- added joint R_ANKLE: type revolute, parent R_LOWER_LEG, child R_FOOT, origin xyz=0 0.0168 -0.30826 rpy=0 0 0, axis 0 1 0, limit lower=-1.6 upper=1.6 effort=1000 velocity=1000
- added joint R_HAA: type revolute, parent R_HIP, child R_SHOULDER, origin xyz=0 0 -0.073 rpy=0 0 0, axis 1 0 0, limit lower=-0.25 upper=0.25 effort=1000 velocity=1000
- added joint R_HFE: type revolute, parent R_SHOULDER, child R_UPPER_LEG, origin xyz=0 0 0 rpy=0 0 0, axis 0 1 0, limit lower=-1.5 upper=1.5 effort=1000 velocity=1000
- added joint R_KFE: type revolute, parent R_UPPER_LEG, child R_LOWER_LEG, origin xyz=0.01 -0.057399 -0.23429 rpy=0 0 0, axis 0 1 0, limit lower=-2.2 upper=-0.1 effort=1000 velocity=1000
- added joint R_YAW: type revolute, parent base_link, child R_HIP, origin xyz=0 -0.0700000000000001 -0.0157999999999999 rpy=0 0 0, axis 0 0 1, limit lower=-0.3 upper=0.3 effort=1000 velocity=1000

Commit message: clean up naming, remove ankle from URDF

File: biped_robot_description/urdf/custom_robot.urdf (robot description, URDF)
Before this commit: robot biped, 12 links, 11 joints
Joints:
- joint L_ANKLE: type revolute -> fixed
- joint R_ANKLE: type revolute -> fixed

Commit message: add foot contact frame, bring back ankle joints, clean up capture point ctrl

File: biped_robot_description/urdf/custom_robot.urdf (robot description, URDF)
Before this commit: robot biped, 12 links, 11 joints
Links:
- added link L_FOOT_CONTACT
- added link R_FOOT_CONTACT
Joints:
- added joint L_FOOT_CONTACT_JOINT: type fixed, parent L_LOWER_LEG, child L_FOOT_CONTACT, origin xyz=0 0.0 -0.32 rpy=0 0 0
- added joint R_FOOT_CONTACT_JOINT: type fixed, parent R_LOWER_LEG, child R_FOOT_CONTACT, origin xyz=0 0.0 -0.32 rpy=0 0 0
- joint L_ANKLE: type fixed -> revolute
- joint R_ANKLE: type fixed -> revolute

Commit message: adjust masses correctly

File: biped_robot_description/urdf/custom_robot.urdf (robot description, URDF)
Before this commit: robot biped, 14 links, 13 joints
Links:
- link base_link: mass 7.62083335132822 -> 6.2

Commit message: put the correct masses & kvs from the sim

File: biped_robot_description/urdf/custom_robot.urdf (robot description, URDF)
Before this commit: robot biped, 14 links, 13 joints
Links:
- link L_SHOULDER: mass 0.588643547253359 -> 1.009
- link L_UPPER_LEG: mass 0.544557667315214 -> 0.8684
- link R_SHOULDER: mass 0.588643548762149 -> 1.009
- link R_UPPER_LEG: mass 0.55166454462452 -> 0.868
- link base_link: mass 2.12328496021261 -> 3.213

Commit message: cleanup xml

File: biped_robot_description/urdf/custom_robot.urdf (robot description, URDF)
Before this commit: robot biped, 14 links, 13 joints
Links:
- link L_LOWER_LEG: mass 0.0923618682215969 -> 0.09236
- link L_UPPER_LEG: mass 0.8684 -> 0.800
- link R_HIP: mass 0.0629568480892821 -> 0.0629568480892822
- link R_LOWER_LEG: mass 0.0923618682215971 -> 0.09236
- link R_UPPER_LEG: mass 0.868 -> 0.800
Joints:
- joint R_KFE: origin xyz=0 -0.0584 -0.23405 rpy=0 0 0 -> xyz=0 -0.0589 -0.23405 rpy=0 0 0

Commit message: new meshes and urdf

File: biped_robot_description/urdf/custom_robot.urdf (robot description, URDF)
Before this commit: robot biped, 14 links, 13 joints
Links:
- link L_FOOT: geometry collision mesh filename=package://biped_robot_description/meshes_v2/L_FOOT.STL; visual mesh filename=package://biped_robot_description/meshes_v2/L_FOOT.STL
- link L_HIP: geometry collision mesh filename=package://biped_robot_description/meshes_v2/L_HIP.STL; visual mesh filename=package://biped_robot_description/meshes_v2/L_HIP.STL
- link L_LOWER_LEG: geometry collision mesh filename=package://biped_robot_description/meshes_v2/L_LOWER_LEG.STL; visual mesh filename=package://biped_robot_description/meshes_v2/L_LOWER_LEG.STL
- link L_SHOULDER: geometry collision mesh filename=package://biped_robot_description/meshes_v2/L_SHOULDER.STL; visual mesh filename=package://biped_robot_description/meshes_v2/L_SHOULDER.STL
- link L_UPPER_LEG: geometry collision mesh filename=package://biped_robot_description/meshes_v2/L_UPPER_LEG.STL; visual mesh filename=package://biped_robot_description/meshes_v2/L_UPPER_LEG.STL
- link R_FOOT: geometry collision mesh filename=package://biped_robot_description/meshes_v2/R_FOOT.STL; visual mesh filename=package://biped_robot_description/meshes_v2/R_FOOT.STL
- link R_HIP: geometry collision mesh filename=package://biped_robot_description/meshes_v2/R_HIP.STL; visual mesh filename=package://biped_robot_description/meshes_v2/R_HIP.STL
- link R_LOWER_LEG: geometry collision mesh filename=package://biped_robot_description/meshes_v2/R_LOWER_LEG.STL; visual mesh filename=package://biped_robot_description/meshes_v2/R_LOWER_LEG.STL
- link R_SHOULDER: geometry collision mesh filename=package://biped_robot_description/meshes_v2/R_SHOULDER.STL; visual mesh filename=package://biped_robot_description/meshes_v2/R_SHOULDER.STL
- link R_UPPER_LEG: geometry collision mesh filename=package://biped_robot_description/meshes_v2/R_UPPER_LEG.STL; visual mesh filename=package://biped_robot_description/meshes_v2/R_UPPER_LEG.STL
- link base_link: geometry collision mesh filename=package://biped_robot_description/meshes_v2/base_link.STL; visual mesh filename=package://biped_robot_description/meshes_v2/base_link.STL

Commit message: urdf to use old meshes and experiment with different feet length

File: biped_robot_description/urdf/custom_robot.urdf (robot description, URDF)
Before this commit: robot biped, 14 links, 13 joints
Links:
- link L_FOOT: geometry collision mesh filename=package://biped_robot_description/meshes/L_FOOT.STL; visual mesh filename=package://biped_robot_description/meshes/L_FOOT.STL
- link L_HIP: geometry collision mesh filename=package://biped_robot_description/meshes/L_HIP.STL; visual mesh filename=package://biped_robot_description/meshes/L_HIP.STL
- link L_LOWER_LEG: geometry collision mesh filename=package://biped_robot_description/meshes/L_LOWER_LEG.STL; visual mesh filename=package://biped_robot_description/meshes/L_LOWER_LEG.STL
- link L_SHOULDER: geometry collision mesh filename=package://biped_robot_description/meshes/L_SHOULDER.STL; visual mesh filename=package://biped_robot_description/meshes/L_SHOULDER.STL
- link L_UPPER_LEG: geometry collision mesh filename=package://biped_robot_description/meshes/L_UPPER_LEG.STL; visual mesh filename=package://biped_robot_description/meshes/L_UPPER_LEG.STL
- link R_FOOT: geometry collision mesh filename=package://biped_robot_description/meshes/R_FOOT.STL; visual mesh filename=package://biped_robot_description/meshes/R_FOOT.STL
- link R_HIP: geometry collision mesh filename=package://biped_robot_description/meshes/R_HIP.STL; visual mesh filename=package://biped_robot_description/meshes/R_HIP.STL
- link R_LOWER_LEG: geometry collision mesh filename=package://biped_robot_description/meshes/R_LOWER_LEG.STL; visual mesh filename=package://biped_robot_description/meshes/R_LOWER_LEG.STL
- link R_SHOULDER: geometry collision mesh filename=package://biped_robot_description/meshes/R_SHOULDER.STL; visual mesh filename=package://biped_robot_description/meshes/R_SHOULDER.STL
- link R_UPPER_LEG: geometry collision mesh filename=package://biped_robot_description/meshes/R_UPPER_LEG.STL; visual mesh filename=package://biped_robot_description/meshes/R_UPPER_LEG.STL
- link base_link: geometry collision mesh filename=package://biped_robot_description/meshes/base_link.STL; visual mesh filename=package://biped_robot_description/meshes/base_link.STL

Commit message: change the limit on vel and effort in urdf

File: biped_robot_description/urdf/custom_robot.urdf (robot description, URDF)
Before this commit: robot biped, 14 links, 13 joints
Joints:
- joint L_ANKLE: limit lower=-1.6 upper=1.6 effort=1000 velocity=1000 -> lower=-1.6 upper=1.6 effort=20 velocity=20
- joint L_HAA: limit lower=-0.25 upper=0.25 effort=1000 velocity=1000 -> lower=-0.25 upper=0.25 effort=20 velocity=20
- joint L_HFE: limit lower=-1.5 upper=1.5 effort=1000 velocity=1000 -> lower=-1.5 upper=1.5 effort=20 velocity=20
- joint L_KFE: limit lower=-2.2 upper=-0.1 effort=1000 velocity=1000 -> lower=-2.2 upper=-0.1 effort=20 velocity=20
- joint L_YAW: limit lower=-0.3 upper=0.3 effort=1000 velocity=1000 -> lower=-0.3 upper=0.3 effort=20 velocity=20
- joint R_ANKLE: limit lower=-1.6 upper=1.6 effort=1000 velocity=1000 -> lower=-1.6 upper=1.6 effort=20 velocity=20
- joint R_HAA: limit lower=-0.25 upper=0.25 effort=1000 velocity=1000 -> lower=-0.25 upper=0.25 effort=20 velocity=20
- joint R_HFE: limit lower=-1.5 upper=1.5 effort=1000 velocity=1000 -> lower=-1.5 upper=1.5 effort=20 velocity=20
- joint R_KFE: limit lower=-2.2 upper=-0.1 effort=1000 velocity=1000 -> lower=-2.2 upper=-0.1 effort=20 velocity=20
- joint R_YAW: limit lower=-0.3 upper=0.3 effort=1000 velocity=1000 -> lower=-0.3 upper=0.3 effort=20 velocity=20
