Commit message: collisions

File: biped_robot_description/urdf/custom_robot_original.urdf (robot description, URDF)
Before this commit: robot biped, 14 links, 13 joints
Links:
- link L_FOOT: geometry collision mesh filename=package://biped_robot_description/meshes/L_FOOT.STL; visual mesh filename=package://biped_robot_description/meshes/L_FOOT.STL
- link R_FOOT: geometry collision mesh filename=package://biped_robot_description/meshes/R_FOOT.STL; visual mesh filename=package://biped_robot_description/meshes/R_FOOT.STL

Commit message: add collision file

File: biped_robot_description/urdf/custom_robot_original.urdf (robot description, URDF)
Before this commit: robot biped, 14 links, 13 joints
Links:
- link base_link: geometry collision mesh filename=package://biped_robot_description/meshes_v3/base_link_colli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; visual mesh filename=package://biped_robot_description/meshes_v3/base_link.STL
