Commit message: add new limits and init

File: biped_robot_description/urdf/custom_robot_v2.urdf (robot description, URDF)
Before this commit: robot biped, 14 links, 13 joints
Joints:
- joint L_KFE: limit lower=-2.2 upper=-0.1 effort=20 velocity=20 -> lower=-2.2 upper=2.2 effort=20 velocity=20
- joint R_KFE: limit lower=-2.2 upper=-0.1 effort=20 velocity=20 -> lower=-2.2 upper=2.2 effort=20 velocity=20

Commit message: fix meshes naming everywhere

File: biped_robot_description/urdf/custom_robot_v2.urdf (robot description, URDF)
Before this commit: robot biped, 14 links, 13 joints
Links:
- link L_HIP: geometry collision mesh filename=package://biped_robot_description/meshes/L_HIP.STL; visual mesh filename=package://biped_robot_description/meshes/L_HIP.STL
- link L_LOWER_LEG: geometry collision mesh filename=package://biped_robot_description/meshes/L_LOWER_LEG.STL; visual mesh filename=package://biped_robot_description/meshes/L_LOWER_LEG.STL
- link L_SHOULDER: geometry collision mesh filename=package://biped_robot_description/meshes/L_SHOULDER.STL; visual mesh filename=package://biped_robot_description/meshes/L_SHOULDER.STL
- link L_UPPER_LEG: geometry collision mesh filename=package://biped_robot_description/meshes/L_UPPER_LEG.STL; visual mesh filename=package://biped_robot_description/meshes/L_UPPER_LEG.STL
- link R_HIP: geometry collision mesh filename=package://biped_robot_description/meshes/R_HIP.STL; visual mesh filename=package://biped_robot_description/meshes/R_HIP.STL
- link R_LOWER_LEG: geometry collision mesh filename=package://biped_robot_description/meshes/R_LOWER_LEG.STL; visual mesh filename=package://biped_robot_description/meshes/R_LOWER_LEG.STL
- link R_SHOULDER: geometry collision mesh filename=package://biped_robot_description/meshes/R_SHOULDER.STL; visual mesh filename=package://biped_robot_description/meshes/R_SHOULDER.STL
- link R_UPPER_LEG: geometry collision mesh filename=package://biped_robot_description/meshes/R_UPPER_LEG.STL; visual mesh filename=package://biped_robot_description/meshes/R_UPPER_LEG.STL
- link base_link: geometry collision mesh filename=package://biped_robot_description/meshes/base_link_v2.STL; visual mesh filename=package://biped_robot_description/meshes/base_link_v2.STL
