Commit message: new URDF for the robot

File: biped_robot_description/urdf/robot_no_yaw.urdf (robot description, URDF)
Before this commit: robot biped, 12 links, 11 joints
Links:
- link L_FOOT: mass 0.046986 -> 0.029476
- link L_LOWER_LEG: mass 0.096474 -> 0.115744
- link L_SHOULDER: mass 0.32272 -> 0.52963
- link L_UPPER_LEG: mass 0.4865 -> 0.958425
- link R_FOOT: mass 0.046986 -> 0.029476
- link R_LOWER_LEG: mass 0.096474 -> 0.11574
- link R_SHOULDER: mass 0.32272 -> 0.52963
- link R_UPPER_LEG: mass 0.47701 -> 0.95843
- link base_link: mass 3.3034 -> 4.8
Joints:
- joint L_HAA: origin xyz=0.005 0.07 -0.090999 rpy=0 0 0 -> xyz=0.005 0.07 -0.091 rpy=0 0 0
- joint L_KFE: origin xyz=0 0.0594 -0.23405 rpy=0 0 0 -> xyz=0 0.0594000000000001 -0.234046496851871 rpy=0 0 0
- joint R_HAA: origin xyz=0.005 -0.07 -0.090999 rpy=0 0 0 -> xyz=0.005 -0.07 -0.091 rpy=0 0 0
